Commit message: Improved collision regions for link_2 and link_3

File: urdf/irb6640_180_255_link_2_geometry.xacro (robot description, xacro)
@@ -6,4 +6,8 @@
 <geometry><box size=".538 1.429 .311" /></geometry>
 </xacro:element>
+<xacro:element xacro:name="${geometry_type}">
+<origin rpy="1.571 0 0"  xyz=".092 -.111 .22" />
+<geometry><box size=".251 .169 .058" /></geometry>
+</xacro:element>
 </xacro:macro>
 </robot>

File: urdf/irb6640_180_255_link_3_geometry.xacro (robot description, xacro)
@@ -11,6 +11,6 @@
 </xacro:element>
 <xacro:element xacro:name="${geometry_type}">
-<origin rpy="0 1.571 0"  xyz=".061 0 .2" />
-<geometry><cylinder length=".35" radius=".166" /></geometry>
+<origin rpy="1.571 0 0"  xyz="0 .018 0" />
+<geometry><cylinder length=".242" radius=".118" /></geometry>
 </xacro:element>
 <xacro:element xacro:name="${geometry_type}">
@@ -19,6 +19,14 @@
 </xacro:element>
 <xacro:element xacro:name="${geometry_type}">
-<origin rpy="1.571 0 0"  xyz="0 .018 0" />
-<geometry><cylinder length=".242" radius=".118" /></geometry>
+<origin rpy="0 1.571 0"  xyz=".061 0 .2" />
+<geometry><cylinder length=".35" radius=".166" /></geometry>
+</xacro:element>
+<xacro:element xacro:name="${geometry_type}">
+<origin rpy="1.571 0 0"  xyz="-.187 -.051 -.029" />
+<geometry><box size=".052 .085 .102" /></geometry>
+</xacro:element>
+<xacro:element xacro:name="${geometry_type}">
+<origin rpy="1.571 0 0"  xyz=".178 -.051 .015" />
+<geometry><box size=".052 .109 .102" /></geometry>
 </xacro:element>
 </xacro:macro>
