Commit message: Fixed issues with dependencies and gazebo launch

File: urdf/irb6640_180_255.xacro (robot description, xacro)
@@ -3,3 +3,8 @@
   <xacro:include filename="$(find rpi_abb_irb6640_180_255_support)/urdf/irb6640_180_255_macro.xacro"/>
   <xacro:abb_irb6640_180_255 prefix=""/>
+  <link name="world"/>
+  <joint name="fixed" type="fixed">
+    <parent link="world"/>
+    <child link="base_link"/>
+  </joint>
 </robot>
